Commit message: Stand_9_6

File: src/bobby/urdf/bobby_gripper_link6.urdf (robot description, URDF)
Before this commit: robot bobby_v3, 12 links, 11 joints
Links:
- link finger_left: geometry collision box size=0.01 0.02 0.09; visual box size=0.01 0.02 0.09
- link finger_right: geometry collision box size=0.01 0.02 0.09; visual box size=0.01 0.02 0.09
- link gripper_base: mass 0.028 -> 0.045; geometry collision box size=0.16 0.03 0.01; visual box size=0.16 0.03 0.01
- link gripper_flange: geometry collision cylinder length=0.01 radius=0.0315; visual cylinder length=0.01 radius=0.0315
- link link_6: geometry 
Joints:
- joint TCP_joint: origin xyz=0 0 0.111 rpy=0 0 0 -> xyz=0 0 0.15 rpy=0 0 0
- joint finger_left_joint: limit lower=0 upper=0.04 effort=50 velocity=0.1 -> lower=0 upper=0.075 effort=50 velocity=0.1; origin xyz=0.006 0 0.021 rpy=0 0 0 -> xyz=0.005 0 0.060000000000000005 rpy=0 0 0
- joint finger_right_joint: limit lower=-0.04 upper=0 effort=50 velocity=0.1 -> lower=-0.075 upper=0 effort=50 velocity=0.1; origin xyz=-0.006 0 0.021 rpy=0 0 0 -> xyz=-0.005 0 0.060000000000000005 rpy=0 0 0
