Commit message: bobby kennt den weg ( fast )

File: src/bobby/urdf/bobby.urdf (robot description, URDF)
Before this commit: robot bobby_v3, 12 links, 11 joints
Joints:
- joint finger_right_joint: mimic joint=finger_left_joint multiplier=-1 offset=0 -> (none)

File: src/scara_robot_pkg/urdf/combined_gazebo.urdf (robot description, URDF)
Before this commit: robot combined_cell, 18 links, 17 joints
Joints:
- joint finger_right_joint: mimic joint=finger_left_joint multiplier=-1 offset=0 -> (none)

File: src/scara_robot_pkg/urdf/drop_box.urdf (robot description, URDF)
Before this commit: robot drop_box, 1 links, 0 joints
Links:
- link drop_box: geometry collision box size=0.02 0.36 0.0188; collision box size=0.02 0.36 0.0188
